File: hardware/logicboard/p2c-000-plain.brd (EAGLE design)
At the start: 91 x 55 mm, 50 parts, among them IC1 74LS07N, K1 G5V1, T1 2SC1815

Commit message: Plain board.
Parts:
- removed A, B: (no value), pinhead:1X04
- removed ANALOG: (no value), con-ml:ML14L
- removed C1: 0.1u, resistor:C025-025X050
- removed C2, C3: 0.01u, resistor:C025-024X044
- removed D1, D2: (no value), SparkFun-DiscreteSemi:DIODE-1N4148
- removed DC12V: POWER_JACKPTH_BREAD, SparkFun-Connectors:POWER_JACK_PTH_BREAD
- removed GND: (no value), SparkFun-Connectors:2X4
- removed I2C: (no value), SparkFun-Connectors:1X05_1MM_RA
- removed IC1: 74LS07N, 74xx-us:DIL14
- removed JP1: (no value), pinhead:2X04
- removed K1: G5V1, relay:G5V1
- removed L1, L2, L3, L4, L5, L6, L7, RCV: (no value), SparkFun-LED:LED_3MM-NS
- removed MIDI: (no value), SparkFun-Connectors:JST-5-PTH
- removed MIDI-IN, MIDI-OUT: DIN5, SparkFun-Connectors:DIN5-RA-PTH
- removed OK1: 6N137, optocoupler:DIL08
- removed PWR2, RST: (no value), SparkFun-Connectors:JST-2-PTH
- removed R1, R2, R3: 220, resistor:0204/5
- removed R4, R5: 10k, resistor:0204/5
- removed R6, R7: 6.8k, resistor:0204/5
- removed RELAY: (no value), SparkFun-Connectors:JST-3-PTH
- removed RN1: 330, resistor-net:RN-9
- removed RN2: 10k, resistor-net:RN-9
- removed SW1: (no value), switch-dil:A1353HEX
- removed T1: 2SC1815, transistor:TO92-ECB
- removed U$2: ARDUINOMICRO, adafruit:ARDUINOMICRO
- removed U$3: KANAYA768_SILK, pineapple:KANAYA768_SILK
- removed U$4: CARDQRCODE450_SILK, pineapple:CARDQRCODE450_SILK
- removed XOUT: (no value), SparkFun-Connectors:1X05
- moved LOGO1 42.6 mm to (45.5, 3.00)
- moved U$1 20.5 mm to (45.5, 50.0)
Connections:
- removed net ANLG_0: ANALOG.2, RN2.2, U$2.P$31
- removed net ANLG_1: ANALOG.4, RN2.3, U$2.P$30
- removed net ANLG_2: ANALOG.6, RN2.4, U$2.P$29
- removed net ANLG_3: ANALOG.8, RN2.5, U$2.P$28
- removed net ANLG_4: ANALOG.10, RN2.6, U$2.P$27
- removed net ANLG_5: ANALOG.12, RN2.7, U$2.P$26
- removed net ANLG_6: ANALOG.14, RN2.8, U$2.P$9
- removed net GND: A.4, C1.2, C2.2, C3.2, DC12V.GND, DC12V.GNDBREAK, DIGITAL.2, GND.1, GND.2, GND.3, GND.4, GND.5, GND.6, GND.7, GND.8, I2C.5, IC1.7, JP1.1, LIGHTDRIVE.2, MIDI-OUT.2, MIDI.2, PWR1.2, PWR2.2, R4.1, RN1.1, RN2.1, RST.2, SW1.C, T1.E, U$2.P$12, U$2.P$21
- removed net I2CENABLE: B.1, JP1.2
- removed net LED1K: L1.K, RN1.2
- removed net LED2K: L2.K, RN1.3
- removed net LED3K: L3.K, RN1.4
- removed net LED4K: L4.K, RN1.5
- removed net LED5K: L5.K, RN1.6
- removed net LED6K: L6.K, RN1.7
- removed net LED7K: L7.K, RN1.8
- removed net MIDIIN: OK1.6, RCV.A, U$2.P$14
- removed net MIDIIN+: MIDI-IN.4, MIDI.4, R3.2
- removed net MIDIIN-: D1.A, MIDI-IN.5, MIDI.5, OK1.3
- removed net MIDIINA: D1.C, OK1.2, R3.1
- removed net MIDIOUT: IC1.1, IC1.11, IC1.13, IC1.3, IC1.5, IC1.9, U$2.P$15
- removed net MIDIOUT+: MIDI-OUT.4, MIDI.1, R2.2
- removed net MIDIOUT-: MIDI-OUT.5, MIDI.3, R1.2
- removed net MIDIOUTC: IC1.2, R1.1
- removed net MOSI: LIGHTDRIVE.7, U$2.P$17
- removed net N$1: RCV.K, RN1.9
- removed net PWM_0: A.3, DIGITAL.9, L1.A, R6.1, U$2.P$10
- removed net PWM_1: DIGITAL.8, L2.A, LIGHTDRIVE.3, U$2.P$8
- removed net PWM_2: DIGITAL.7, L3.A, U$2.P$7
- removed net PWM_3: DIGITAL.6, L4.A, U$2.P$4
- removed net PWM_4: DIGITAL.5, L5.A, U$2.P$3
- removed net PWM_5: DIGITAL.4, L6.A, U$2.P$2
- removed net PWM_6: DIGITAL.3, JP1.8, L7.A, U$2.P$34
- removed net RELAYCOM: K1.5, K1.6, RELAY.2
- removed net RELAYDRIVE: R4.2, R5.1, T1.B
- removed net RELAYNC: K1.1, RELAY.3
- removed net RELAYNO: K1.10, RELAY.1
- removed net RELAYTR: D2.A, K1.9, T1.C
- removed net RLYDRV: JP1.7, R5.2
- removed net RST: RST.1, U$2.P$22
- removed net SCL: B.3, I2C.3
- removed net SCLK: LIGHTDRIVE.6, U$2.P$18
- removed net SDA: B.2, I2C.4
- removed net SW0: JP1.3, SW1.1
- removed net SW1: JP1.5, SW1.2
- removed net SW_0: A.2, JP1.4, R7.1, U$2.P$11
- removed net SW_1: I2C.2, JP1.6, U$2.P$6
- removed net SW_2: LIGHTDRIVE.4, SW1.4, U$2.P$5
- removed net SW_3: LIGHTDRIVE.5, SW1.8, U$2.P$1
- removed net VCC: A.1, ANALOG.1, ANALOG.11, ANALOG.13, ANALOG.3, ANALOG.5, ANALOG.7, ANALOG.9, C1.1, C2.1, C3.1, D2.C, IC1.14, K1.2, LIGHTDRIVE.1, OK1.7, R2.1, R6.2, R7.2, U$2.P$23
- removed net VDD: B.4, DIGITAL.1, I2C.1, U$2.P$33
- removed net VIN: DC12V.PWR, PWR1.1, PWR2.1, U$2.P$20
- removed net X1: IC1.4, XOUT.1
- removed net X2: IC1.6, XOUT.2
- removed net X3: IC1.8, XOUT.3
- removed net X4: IC1.10, XOUT.4
- removed net X5: IC1.12, XOUT.5
Routing:
- net GND: track 344.6 -> 0.00 mm, vias 1 -> 0
- net VCC: track 179.2 -> 0.00 mm, vias 2 -> 0
- net PWM_1: track 173.0 -> 0.00 mm, vias 2 -> 0
- net VDD: track 149.7 -> 0.00 mm, vias 6 -> 0
- net PWM_6: track 149.0 -> 0.00 mm, vias 4 -> 0
- net PWM_0: track 136.0 -> 0.00 mm, vias 1 -> 0
- net SW_1: track 120.5 -> 0.00 mm, vias 3 -> 0
- net ANLG_1: track 118.2 -> 0.00 mm, vias 1 -> 0
- net ANLG_2: track 112.1 -> 0.00 mm, vias 4 -> 0
- net ANLG_0: track 105.3 -> 0.00 mm, vias 4 -> 0
- net ANLG_6: track 105.2 -> 0.00 mm, vias 5 -> 0
- net SW_3: track 86.6 -> 0.00 mm
- net PWM_5: track 84.5 -> 0.00 mm, vias 1 -> 0
- net SW_2: track 82.2 -> 0.00 mm, vias 2 -> 0
- net ANLG_4: track 81.7 -> 0.00 mm, vias 3 -> 0
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Other:
- board text removed: "3"
- board text removed: "4"
- board text removed: "5"
- board text removed: "A0"
- board text removed: "A1"
- board text removed: "A2"
- board text removed: "A3"
- board text removed: "A4"
- board text removed: "A5"
- board text removed: "A6"
- board text removed: "ANALOG"
- board text removed: "Com."
- board text removed: "D2"
- board text removed: "D7"
- board text removed: "Founder, Pineapple Computer Founder, TEDxSaikai Professor, Univ. of Nagasaki https://pineapple.cc/card kanaya@pineapple.cc, @kanaya"
- board text removed: "G"
- board text removed: "How to make"
- board text removed: "IC2"
- board text removed: "IN"
- board text removed: "Ichi KANAYA, Ph.D."
- board text removed: "MC1"
- board text removed: "MC1: Arduino Micro 5V SW1: Comp. HEX Con 5V: Pin 2p Con Analog: ML 14p Con DC: DC Jack Con Digital: Pin 9p Con GND: Pin 2x4p Con Lightdrive: Pin 7p Con I2C: SH 5p Con MIDI: DIN 5p/PH 5p Con Relay: PH 3p Con RST: PH 2p Con XOUT: Pin 5p Pogo: Pin 1p"
- board text removed: "N.C."
- board text removed: "N.O."
- board text removed: "NC"
- board text removed: "OUT"
- board text removed: "Pineapple IIc 1.2.0"
- board text removed: "R1-3: 220 R4-5: 10k R6-7: 6.8k RN1: 330 RN2: 10k C1: 0.1u C2-3: 0.01u K1: G5V-1 D1-2: 1N4148 LED1-8: If20m T1: 2SC1815 OK1: TLP552 IC1: 74LS07 IC2: PCA9517ADP"
- board text removed: "USB>>"

Commit message: Plain board.
Connections:
- new net GND: DIGITAL.2, LIGHTDRIVE.2, PWR1.2
Changed lines of the file:
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@@
 <vertex x="-2" y="57"/>
 </polygon>
+<contactref element="PWR1" pad="2"/>
+<contactref element="DIGITAL" pad="2"/>
+<contactref element="LIGHTDRIVE" pad="2"/>
+<wire x1="11.43" y1="3" x2="80.01" y2="3" width="0" layer="19" extent="1-1"/>
+<wire x1="11.43" y1="51.26" x2="11.43" y2="3" width="0" layer="19" extent="1-1"/>
 </signal>
 </signals>
