File: hardware/logicboard/p2c-000-plain.sch (EAGLE design)
At the start: 50 parts, among them IC1 74LS07N, K1 G5V1, T1 2SC1815

Commit message: Plain board.
Parts:
- removed A, B: (no value), pinhead:PINHD-1X4
- removed ANALOG: (no value), con-ml:ML14L
- removed C1: 0.1u, resistor:C-US025-025X050
- removed C2, C3: 0.01u, resistor:C-US025-024X044
- removed D1, D2: DIODE-1N4148, SparkFun-DiscreteSemi:DIODE-1N4148
- removed DC12V: POWER_JACKPTH_BREAD, SparkFun-Connectors:POWER_JACKPTH_BREAD
- removed GND: (no value), SparkFun-Connectors:CONN_04X2
- removed I2C: (no value), SparkFun-Connectors:CONN_05SMD2
- removed IC1: 74LS07N, 74xx-us:74LS07N
- removed JP1: (no value), pinhead:PINHD-2X4
- removed K1: G5V1, relay:G5V1
- removed L1, L2, L3, L4, L5, L6, L7, RCV: (no value), SparkFun-LED:LED-3MM-NO_SILK
- removed MIDI: (no value), SparkFun-Connectors:CONN_05JST
- removed MIDI-IN, MIDI-OUT: DIN5, SparkFun-Connectors:DIN5
- removed OK1: 6N137, optocoupler:6N137
- removed PWR2, RST: (no value), SparkFun-Connectors:CONN_02JST-PTH-2
- removed R1, R2, R3: 220, resistor:R-US_0204/5
- removed R4, R5: 10k, resistor:R-US_0204/5
- removed R6, R7: 6.8k, resistor:R-US_0204/5
- removed RELAY: (no value), SparkFun-Connectors:CONN_03JST-PTH
- removed RN1: 330, resistor-net:RN08
- removed RN2: 10k, resistor-net:RN08
- removed SW1: (no value), switch-dil:A1353HEX
- removed T1: 2SC1815, transistor:2SC1815
- removed U$2: ARDUINOMICRO, adafruit:ARDUINOMICRO
- removed U$3: KANAYA768_SILK, pineapple:KANAYA768_SILK
- removed U$4: CARDQRCODE450_SILK, pineapple:CARDQRCODE450_SILK
- removed XOUT: (no value), SparkFun-Connectors:CONN_05
Connections:
- removed net ANLG_0: ANALOG.2, RN2.2, U$2.A0
- removed net ANLG_1: ANALOG.4, RN2.3, U$2.A1
- removed net ANLG_2: ANALOG.6, RN2.4, U$2.A2
- removed net ANLG_3: ANALOG.8, RN2.5, U$2.A3
- removed net ANLG_4: ANALOG.10, RN2.6, U$2.A4
- removed net ANLG_5: ANALOG.12, RN2.7, U$2.A5
- removed net ANLG_6: ANALOG.14, RN2.8, U$2.4
- removed net GND: A.4, C1.2, C2.2, C3.2, DC12V.GND, DC12V.GNDBREAK, DIGITAL.2, GND.1, GND.2, GND.3, GND.4, GND.5, GND.6, GND.7, GND.8, I2C.5, JP1.1, LIGHTDRIVE.2, MIDI-OUT.2, MIDI.2, PWR1.2, PWR2.2, R4.1, RN1.1, RN2.1, RST.2, SW1.C, T1.E, U$2.GND, U$2.GND@1
- removed net I2CENABLE: B.1, JP1.2
- removed net LED1K: L1.C, RN1.2
- removed net LED2K: L2.C, RN1.3
- removed net LED3K: L3.C, RN1.4
- removed net LED4K: L4.C, RN1.5
- removed net LED5K: L5.C, RN1.6
- removed net LED6K: L6.C, RN1.7
- removed net LED7K: L7.C, RN1.8
- removed net MIDIIN: OK1.VO, RCV.A, U$2.RX
- removed net MIDIIN+: MIDI-IN.4, MIDI.4, R3.2
- removed net MIDIIN-: D1.A, MIDI-IN.5, MIDI.5, OK1.C
- removed net MIDIINA: D1.C, OK1.A, R3.1
- removed net MIDIOUT: IC1A.I, IC1B.I, IC1C.I, IC1D.I, IC1E.I, IC1F.I, U$2.TX
- removed net MIDIOUT+: MIDI-OUT.4, MIDI.1, R2.2
- removed net MIDIOUT-: MIDI-OUT.5, MIDI.3, R1.2
- removed net MIDIOUTC: IC1A.O, R1.1
- removed net MOSI: LIGHTDRIVE.7, U$2.MOSI
- removed net N$1: RCV.C, RN1.9
- removed net PWM_0: A.3, DIGITAL.9, L1.A, R6.1, U$2.3
- removed net PWM_1: DIGITAL.8, L2.A, LIGHTDRIVE.3, U$2.5
- removed net PWM_2: DIGITAL.7, L3.A, U$2.6
- removed net PWM_3: DIGITAL.6, L4.A, U$2.9
- removed net PWM_4: DIGITAL.5, L5.A, U$2.10
- removed net PWM_5: DIGITAL.4, L6.A, U$2.11
- removed net PWM_6: DIGITAL.3, JP1.8, L7.A, U$2.13
- removed net RELAYCOM: K12.P, K12.P@1, RELAY.2
- removed net RELAYDRIVE: R4.2, R5.1, T1.B
- removed net RELAYNC: K12.O, RELAY.3
- removed net RELAYNO: K12.S, RELAY.1
- removed net RELAYTR: D2.A, K11.2, T1.C
- removed net RLYDRV: JP1.7, R5.2
- removed net RST: RST.1, U$2.R@2
- removed net SCL: B.3, I2C.3
- removed net SCLK: LIGHTDRIVE.6, U$2.SCK
- removed net SDA: B.2, I2C.4
- removed net SW0: JP1.3, SW1.1
- removed net SW1: JP1.5, SW1.2
- removed net SW_0: A.2, JP1.4, R7.1, U$2.2
- removed net SW_1: I2C.2, JP1.6, U$2.7
- removed net SW_2: LIGHTDRIVE.4, SW1.4, U$2.8
- removed net SW_3: LIGHTDRIVE.5, SW1.8, U$2.12
- removed net VCC: A.1, ANALOG.1, ANALOG.11, ANALOG.13, ANALOG.3, ANALOG.5, ANALOG.7, ANALOG.9, C1.1, C2.1, C3.1, D2.C, K11.1, LIGHTDRIVE.1, OK1.VE, R2.1, R6.2, R7.2, U$2.5V
- removed net VDD: B.4, DIGITAL.1, I2C.1, U$2.3V
- removed net VIN: DC12V.PWR, PWR1.1, PWR2.1, U$2.9V
- removed net X1: IC1B.O, XOUT.1
- removed net X2: IC1C.O, XOUT.2
- removed net X3: IC1D.O, XOUT.3
- removed net X4: IC1E.O, XOUT.4
- removed net X5: IC1F.O, XOUT.5
Other:
- moved on the sheet: DIGITAL, LIGHTDRIVE, POGOPIN, PWR1

Commit message: Plain board.
Connections:
- new net GND: DIGITAL.2, LIGHTDRIVE.2, PWR1.2
Other:
- moved on the sheet: LIGHTDRIVE, POGOPIN
Changed lines of the file:
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@@
 <part name="POGOPIN" library="pinhead" library_urn="urn:adsk.eagle:library:325" deviceset="PINHD-1X1" device="" package3d_urn="urn:adsk.eagle:package:22485/2"/>
 <part name="PWR1" library="SparkFun-Connectors" library_urn="urn:adsk.eagle:library:513" deviceset="CONN_02" device="" package3d_urn="urn:adsk.eagle:package:38039/1"/>
+<part name="SUPPLY1" library="supply2" library_urn="urn:adsk.eagle:library:372" deviceset="GND" device=""/>
+<part name="SUPPLY2" library="supply2" library_urn="urn:adsk.eagle:library:372" deviceset="GND" device=""/>
+<part name="SUPPLY3" library="supply2" library_urn="urn:adsk.eagle:library:372" deviceset="GND" device=""/>
 </parts>
 <sheets>
@@
 <instance part="LOGO1" gate="G$1" x="241.3" y="165.1"/>
 <instance part="DIGITAL" gate="G$1" x="7.62" y="147.32" rot="MR180"/>
-<instance part="LIGHTDRIVE" gate="G$1" x="12.7" y="121.92" rot="MR180"/>
-<instance part="POGOPIN" gate="G$1" x="12.7" y="101.6"/>
+<instance part="LIGHTDRIVE" gate="G$1" x="12.7" y="119.38" rot="MR180"/>
+<instance part="POGOPIN" gate="G$1" x="226.06" y="167.64"/>
 <instance part="PWR1" gate="G$1" x="10.16" y="170.18" rot="MR180"/>
+<instance part="SUPPLY1" gate="GND" x="20.32" y="162.56"/>
+<instance part="SUPPLY2" gate="GND" x="20.32" y="132.08"/>
+<instance part="SUPPLY3" gate="GND" x="20.32" y="101.6"/>
 </instances>
 <busses>
 </busses>
 <nets>
+<net name="GND" class="0">
+<segment>
+<pinref part="PWR1" gate="G$1" pin="2"/>
+<pinref part="SUPPLY1" gate="GND" pin="GND"/>
+<wire x1="17.78" y1="167.64" x2="20.32" y2="167.64" width="0.1524" layer="91"/>
+<wire x1="20.32" y1="167.64" x2="20.32" y2="165.1" width="0.1524" layer="91"/>
+</segment>
+<segment>
+<pinref part="DIGITAL" gate="G$1" pin="2"/>
+<pinref part="SUPPLY2" gate="GND" pin="GND"/>
+<wire x1="17.78" y1="154.94" x2="20.32" y2="154.94" width="0.1524" layer="91"/>
+<wire x1="20.32" y1="154.94" x2="20.32" y2="134.62" width="0.1524" layer="91"/>
+</segment>
+<segment>
+<pinref part="LIGHTDRIVE" gate="G$1" pin="2"/>
+<pinref part="SUPPLY3" gate="GND" pin="GND"/>
+<wire x1="17.78" y1="121.92" x2="20.32" y2="121.92" width="0.1524" layer="91"/>
+<wire x1="20.32" y1="121.92" x2="20.32" y2="104.14" width="0.1524" layer="91"/>
+</segment>
+</net>
 </nets>
 </sheet>
